File: Boards/SirMicro/SirMicro3V3/SirMicro3V3.sch (KiCad schematic (older format))
At the start: 32 parts, among them J1 Conn_01x16, J2 Conn_01x16, J3 USB_B_Micro, U1 ATmega32U4-AU, U2 AP2127K-3.3, Y1 Resonator

Commit message: Board Layout revised and 3V3 Version Added
Connections:
- net 3V3: now also C1.1, C4.1, C5.1, C7.1, D1.1 (K), ICSP6.2 (Pin_2), J1.2 (Pin_2), JP1.1 (A), L1.1, R3.1, RN1.2 (R2.1), U1.14 (VCC), U1.2 (UVCC), U1.34 (VCC), U1.6 (UCAP), U1.7 (VBUS)
- net 5V: no longer C1.1, C4.1, C5.1, C7.1, D1.1 (K), ICSP6.2 (Pin_2), J1.2 (Pin_2), JP1.1 (A), L1.1, R3.1, RN1.2 (R2.1), U1.14 (VCC), U1.2 (UVCC), U1.34 (VCC), U1.6 (UCAP), U1.7 (VBUS)
Changed lines of the file:
@@
 EESchema Schematic File Version 4
-LIBS:SirMicro5V-cache
+LIBS:SirMicro3V3-cache
 EELAYER 29 0
 EELAYER END
@@
 Wire Wire Line
 	2000 3250 1950 3250
-Wire Wire Line
-	2000 2600 2000 1450
 Connection ~ 2750 1450
 Wire Wire Line
@@
 Wire Wire Line
 	2550 2300 2750 2300
-Connection ~ 2550 1450
 Wire Wire Line
 	2550 1450 2750 1450
-Wire Wire Line
-	2000 1450 2550 1450
 $Comp
 L Device:CP C8
@@
 Wire Wire Line
 	2550 2300 2550 2750
-Text GLabel 2000 1450 0    50   Input ~ 0
+Text GLabel 2000 2500 0    50   Input ~ 0
 5V
 Text GLabel 8750 1600 2    50   Input ~ 0
@@
 Wire Wire Line
 	8400 4550 8300 4550
-Text GLabel 8400 4650 2    50   Input ~ 0
-5V
 Wire Wire Line
 	8400 4650 8300 4650
@@
 Wire Wire Line
 	5850 1800 6000 1800
-Text GLabel 6600 1600 2    50   Input ~ 0
-5V
 Text GLabel 6600 1800 2    50   Input ~ 0
 GND
@@
 D13
 Text GLabel 7250 3100 0    50   Input ~ 0
-5V
+3V3
 Wire Wire Line
 	8050 2000 8450 2000
@@
 Connection ~ 3550 3050
 Text GLabel 2650 3050 0    50   Input ~ 0
-5V
+3V3
 Wire Wire Line
 	2650 3050 2850 3050
+Wire Wire Line
+	2000 2600 2000 2500
+Text GLabel 5100 1450 2    50   Input ~ 0
+3V3
+Text GLabel 6600 1600 2    50   Input ~ 0
+3V3
+Text GLabel 8400 4650 2    50   Input ~ 0
+3V3
 $EndSCHEMATC
