File: Boards/SirIoT/SIM28ML/SIM28ML.kicad_pcb (KiCad board)
At the start: 2 copper layers, 22.7 x 20.3 mm, 26 parts, among them J1 Conn_01x05, J2 Conn_01x05, U2 AP7365-W-7

Commit message: GNSS Boards Page Layout Updates
Parts:
- renumbered SIM28M to SIM28ML
Other:
- board text added: "SIM28ML www.SirBoard.com"
- board text removed: "SIM28M www.SirBoard.com"
Changed lines of the file:
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@@
   (page User 132.004 102.006)
   (title_block
-    (title "SIM28M Based GPS Module")
+    (title "SIM28ML Based GPS Module")
     (date 2019-10-30)
     (rev 1)
     (company SirBoard)
-    (comment 1 "SIM28M is based on the MT3339 Chipset")
+    (comment 1 "SIM28ML is based on the MT3339 Chipset")
     (comment 2 "Breadboard Friendly Micro GPS Module")
   )
@@
     (tags "Integrated Circuit")
     (attr smd)
-    (fp_text reference SIM28M (at 4.85 5.05 90) (layer F.SilkS)
+    (fp_text reference SIM28ML (at 4.85 5.05 90) (layer F.SilkS)
       (effects (font (size 1.27 1.27) (thickness 0.254)))
     )
@@
     )
   )
-  (gr_text "SIM28M\nwww.SirBoard.com" (at 63.5 31.242 180) (layer B.SilkS)
+  (gr_text "SIM28ML\nwww.SirBoard.com" (at 63.5 31.242 180) (layer B.SilkS)
     (effects (font (size 1 0.9) (thickness 0.15)) (justify mirror))
   )
