File: Modules/SirKeep/MB85RCXXX/MB85RCXXX.kicad_pcb (KiCad board)
At the start: 2 copper layers, 18 x 16.8 mm, 17 parts, among them J1 Conn_01x05

Commit message: MB85RXXX Added in place of MB85RC256V
Parts:
- G***: footprint logo:logo76x107 -> logo:logo63x89
- moved G*** 2.17 mm to (59.1, 46.6)
- moved G*** 0.38 mm to (53.5, 44.8)
Other:
- board text added: "128kB"
- board text added: "16kB"
- board text added: "32kB"
- board text added: "64kB"
- board text added: "8kB"
- board text added: "MB85RCXXX I2C FRAM"
- board text removed: "MB85RC256V I2C FRAM 32kBytes"
