File: Boards/SirUSB/CP2102/CP2102.kicad_pcb (KiCad board)
At the start: 2 copper layers, 20.7 x 15.5 mm, 23 parts, among them J1 USB_B_Micro, J2 Conn_01x03, J3 Conn_01x03, J4 Conn_01x06, U1 FT231XQ

Commit message: Soldermask width adjusted
Other:
- rule solder_mask_min_width: 0.05 -> 0.1
Changed lines of the file:
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@@
     (pad_drill 1)
     (pad_to_mask_clearance 0)
-    (solder_mask_min_width 0.05)
+    (solder_mask_min_width 0.1)
     (aux_axis_origin 0 0)
     (visible_elements 7FFFFFFF)
